Commit message: Update names, credits and the README for the new layout
- Rename armbot to conveysort inside the files, so the package names,
  the robot's name and the paths match the new folders.
- Credit the borrowed code: Antonio Brandi's course (Apache-2.0, with
  LICENSE-APACHE and a notice in each file), Ujwal Nandanwar's ESP32
  sketch (MIT) and the ROS 2 docs' dev container guide (CC BY 4.0).
- Read the ESP32 access point's password from a git-ignored secrets.h.
- Use the GitHub noreply address as maintainer, and Apache-2.0 as the
  licence name in every package.
- Remove three meshes nothing uses.
- Put run-container.sh's shebang on its first line; keep the executable
  bit on shell scripts only.
- Write the README and experiments/README.md, with photos and videos.

Co-Authored-By: Claude Opus 5.5 <noreply@anthropic.com>

File: src/conveysort_description/urdf/conveysort_arm.urdf.xacro (robot description, xacro)
@@ -1,10 +1,16 @@
 <?xml version="1.0"?>
-<robot xmlns:xacro="http://www.ros.org/wiki/xacro" name="armbot">
+<!--
+  ConveySort-Arm's model. The arm's links, joints and meshes come from my team's EnviroBot project
+  (https://github.com/jewel-nath/envirobot). The file's layout follows the arduinobot code from
+  Antonio Brandi's course "Robotics and ROS 2 - Learn by Doing! Manipulators"
+  (https://github.com/AntoBrandi/Robotics-and-ROS-2-Learn-by-Doing-Manipulators), Apache License 2.0 (LICENSE-APACHE).
+-->
+<robot xmlns:xacro="http://www.ros.org/wiki/xacro" name="conveysort_arm">
     <!-- Load Simulated or Real Hardware Interfaces -->
     <xacro:arg name="is_sim" default="true"/>
     <!-- Include Gazebo Parameters -->
-    <xacro:include filename="$(find armbot_description)/urdf/armbot_gazebo.xacro" />
+    <xacro:include filename="$(find conveysort_description)/urdf/conveysort_arm_gazebo.xacro" />
     <!-- Include ros2_control Plugins -->
-    <xacro:include filename="$(find armbot_description)/urdf/armbot_ros2_control.xacro" />
+    <xacro:include filename="$(find conveysort_description)/urdf/conveysort_arm_ros2_control.xacro" />
     <!-- Useful XACRO Variables (Properties) -->
     <xacro:property name="PI" value="3.14159265359" />
@@ -37,5 +43,5 @@
             <origin rpy="0 0 0" xyz="0 0 0.01" />
             <geometry>
-                <mesh filename="package://armbot_description/meshes/base_cylinder.stl"
+                <mesh filename="package://conveysort_description/meshes/base_cylinder.stl"
                     scale="0.0001 0.0001 0.0001" />
             </geometry>
@@ -47,5 +53,5 @@
             <origin rpy="0 0 0" xyz="0 0 0.01" />
             <geometry>
-                <mesh filename="package://armbot_description/meshes/base_cylinder.stl"
+                <mesh filename="package://conveysort_description/meshes/base_cylinder.stl"
                     scale="0.0001 0.0001 0.0001" />
             </geometry>
@@ -57,13 +63,13 @@
             <origin rpy="0 0 0" xyz="0 0 0" />
             <geometry>
-                <mesh filename="package://armbot_description/meshes/top_plate.stl"
-                    scale="0.001 0.001 0.001" />
-            </geometry>
-            <material name="black" />
-        </visual>
-        <collision>
-            <origin rpy="0 0 0" xyz="0 0 0" />
-            <geometry>
-                <mesh filename="package://armbot_description/meshes/top_plate.stl"
+                <mesh filename="package://conveysort_description/meshes/top_plate.stl"
+                    scale="0.001 0.001 0.001" />
+            </geometry>
+            <material name="black" />
+        </visual>
+        <collision>
+            <origin rpy="0 0 0" xyz="0 0 0" />
+            <geometry>
+                <mesh filename="package://conveysort_description/meshes/top_plate.stl"
                     scale="0.001 0.001 0.001" />
             </geometry>
@@ -75,13 +81,13 @@
             <origin rpy="0 0 0" xyz="0 0 0" />
             <geometry>
-                <mesh filename="package://armbot_description/meshes/lower_arm.stl"
-                    scale="0.001 0.001 0.001" />
-            </geometry>
-            <material name="black" />
-        </visual>
-        <collision>
-            <origin rpy="0 0 0" xyz="0 0 0" />
-            <geometry>
-                <mesh filename="package://armbot_description/meshes/lower_arm.stl"
+                <mesh filename="package://conveysort_description/meshes/lower_arm.stl"
+                    scale="0.001 0.001 0.001" />
+            </geometry>
+            <material name="black" />
+        </visual>
+        <collision>
+            <origin rpy="0 0 0" xyz="0 0 0" />
+            <geometry>
+                <mesh filename="package://conveysort_description/meshes/lower_arm.stl"
                     scale="0.001 0.001 0.001" />
             </geometry>
@@ -93,5 +99,5 @@
             <origin rpy="0 1.59 0" xyz="0 0 0" />
             <geometry>
-                <mesh filename="package://armbot_description/meshes/top_arm.stl"
+                <mesh filename="package://conveysort_description/meshes/top_arm.stl"
                     scale="0.001 0.001 0.001" />
             </geometry>
@@ -101,5 +107,5 @@
             <origin rpy="0 1.59 0" xyz="0 0 0" />
             <geometry>
-                <mesh filename="package://armbot_description/meshes/top_arm.stl"
+                <mesh filename="package://conveysort_description/meshes/top_arm.stl"
                     scale="0.001 0.001 0.001" />
             </geometry>
@@ -111,13 +117,13 @@
             <origin rpy="0 0 0" xyz="0 0 0" />
             <geometry>
-                <mesh filename="package://armbot_description/meshes/wrist.stl"
-                    scale="0.001 0.001 0.001" />
-            </geometry>
-            <material name="black" />
-        </visual>
-        <collision>
-            <origin rpy="0 0 0" xyz="0 0 0" />
-            <geometry>
-                <mesh filename="package://armbot_description/meshes/wrist.stl"
+                <mesh filename="package://conveysort_description/meshes/wrist.stl"
+                    scale="0.001 0.001 0.001" />
+            </geometry>
+            <material name="black" />
+        </visual>
+        <collision>
+            <origin rpy="0 0 0" xyz="0 0 0" />
+            <geometry>
+                <mesh filename="package://conveysort_description/meshes/wrist.stl"
                     scale="0.001 0.001 0.001" />
             </geometry>
@@ -129,5 +135,5 @@
             <origin rpy="0 3.18 0" xyz="0 0 0" />
             <geometry>
-                <mesh filename="package://armbot_description/meshes/clawbase.stl"
+                <mesh filename="package://conveysort_description/meshes/clawbase.stl"
                     scale="0.001 0.001 0.001" />
             </geometry>
@@ -139,5 +145,5 @@
             <origin rpy="0 3.18 0" xyz="0 0 0" />
             <geometry>
-                <mesh filename="package://armbot_description/meshes/clawbase.stl"
+                <mesh filename="package://conveysort_description/meshes/clawbase.stl"
                     scale="0.001 0.001 0.001" />
             </geometry>
@@ -149,5 +155,5 @@
             <origin rpy="0 0 0" xyz="0 0 0" />
             <geometry>
-                <mesh filename="package://armbot_description/meshes/clawr.stl"
+                <mesh filename="package://conveysort_description/meshes/clawr.stl"
                     scale="0.001 0.001 0.001" />
             </geometry>
@@ -157,5 +163,5 @@
             <origin rpy="0 0 0" xyz="0 0 0" />
             <geometry>
-                <mesh filename="package://armbot_description/meshes/clawr.stl"
+                <mesh filename="package://conveysort_description/meshes/clawr.stl"
                     scale="0.001 0.001 0.001" />
             </geometry>
@@ -167,5 +173,5 @@
             <origin rpy="0 0 0" xyz="0 0 0" />
             <geometry>
-                <mesh filename="package://armbot_description/meshes/clawl.stl"
+                <mesh filename="package://conveysort_description/meshes/clawl.stl"
                     scale="0.001 0.001 0.001" />
             </geometry>
@@ -175,5 +181,5 @@
             <origin rpy="0 0 0" xyz="0 0 0" />
             <geometry>
-                <mesh filename="package://armbot_description/meshes/clawl.stl"
+                <mesh filename="package://conveysort_description/meshes/clawl.stl"
                     scale="0.001 0.001 0.001" />
             </geometry>

File: src/conveysort_description/urdf/conveysort_arm_gazebo.xacro (robot description, xacro)
@@ -1,4 +1,10 @@
 <?xml version="1.0"?>
-<robot xmlns:xacro="http://www.ros.org/wiki/xacro" name="armbot">
+<!--
+  Based on the arduinobot code from Antonio Brandi's course "Robotics and ROS 2 - Learn by Doing!
+  Manipulators": https://github.com/AntoBrandi/Robotics-and-ROS-2-Learn-by-Doing-Manipulators
+  Licensed under the Apache License 2.0 (LICENSE-APACHE). Changed for ConveySort-Arm: the names,
+  and in some files the arm's joints and servos.
+-->
+<robot xmlns:xacro="http://www.ros.org/wiki/xacro" name="conveysort_arm">
     <!-- Gazebo ros2_control plugin -->
     <gazebo>
@@ -6,5 +12,5 @@
         <robot_param>robot_description</robot_param>
         <robot_param_node>robot_state_publisher</robot_param_node>
-        <parameters>$(find armbot_controller)/config/armbot_controllers.yaml</parameters>
+        <parameters>$(find conveysort_controller)/config/conveysort_arm_controllers.yaml</parameters>
       </plugin>
     </gazebo>

File: src/conveysort_description/urdf/conveysort_arm_ros2_control.xacro (robot description, xacro)
@@ -1,4 +1,10 @@
 <?xml version="1.0"?>
-<robot xmlns:xacro="http://www.ros.org/wiki/xacro" name="armbot">
+<!--
+  Based on the arduinobot code from Antonio Brandi's course "Robotics and ROS 2 - Learn by Doing!
+  Manipulators": https://github.com/AntoBrandi/Robotics-and-ROS-2-Learn-by-Doing-Manipulators
+  Licensed under the Apache License 2.0 (LICENSE-APACHE). Changed for ConveySort-Arm: the names,
+  and in some files the arm's joints and servos.
+-->
+<robot xmlns:xacro="http://www.ros.org/wiki/xacro" name="conveysort_arm">
     <ros2_control name="RobotSystem" type="system">
         <xacro:property name="PI" value="3.14159265359" />
@@ -9,5 +15,5 @@
             </hardware>
             <hardware>
-                <plugin>armbot_controller/ArmbotInterface</plugin>
+                <plugin>conveysort_controller/ConveysortInterface</plugin>
                 <param name="port">/dev/ttyACM0</param>
             </hardware>
@@ -24,5 +30,5 @@
         <xacro:unless value="$(arg is_sim)">
             <hardware>
-                <plugin>armbot_controller/ArmbotInterface</plugin>
+                <plugin>conveysort_controller/ConveysortInterface</plugin>
                 <param name="port">/dev/ttyACM0</param>
             </hardware>
